File: kicad/amosis.kicad_pcb (KiCad board)
At the start: 2 copper layers, 60 x 90 mm, 87 parts, among them J1 USB-C-16, J2 USB-C-16, J3 VALVE, M1 GND, M2 GND, M3 GND, Q1 MMBT3904, SW22 RESET, SW23 BOOT, U1 MIC5504-3.3YM5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

Commit message: logic & fixes
Parts:
- D25, D26: value CESD5V0D5 -> DESD5V0U1BA
- tRUN1: value RUN -> VCC
- moved COL_{0}1 30.0 mm to (15.0, 5.00)
- moved COL_{6}1 30.0 mm to (-15.0, 5.00)
- moved COL_{1}1 20.0 mm to (10.0, 5.00)
- moved COL_{5}1 20.0 mm to (-10.0, 5.00)
- moved COL_{2}1 10.0 mm to (5.00, 5.00)
- moved COL_{4}1 10.0 mm to (-5.00, 5.00)
Connections:
- U3 pad 15: /COL_{0} -> /COL_{6}
- U3 pad 16: /COL_{1} -> /COL_{5}
- U3 pad 17: /COL_{2} -> /COL_{4}
- U3 pad 27: /COL_{4} -> /COL_{2}
- U3 pad 28: /COL_{5} -> /COL_{1}
- U3 pad 29: /COL_{6} -> /COL_{0}
Routing:
- net /COL_{6}: track 26.7 -> 32.9 mm
- net /COL_{0}: track 32.9 -> 26.7 mm
- net /COL_{5}: track 26.6 -> 30.9 mm
- net /COL_{1}: track 30.9 -> 26.6 mm
Changed lines of the file:
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@@
 	(footprint "fp:PinHeader_1x01"
 		(layer "F.Cu")
-		(at 10 5)
+		(at -10 5)
 		(descr "Through hole straight pin header, 1x03, 1.00mm pitch, single row")
 		(tags "Through hole pin header THT 1x03 1.00mm single row")
@@
 	(footprint "fp:PinHeader_1x01"
 		(layer "F.Cu")
-		(at 5 5)
+		(at -5 5)
 		(descr "Through hole straight pin header, 1x03, 1.00mm pitch, single row")
 		(tags "Through hole pin header THT 1x03 1.00mm single row")
@@
 			)
 		)
-		(property "Value" "CESD5V0D5"
+		(property "Value" "DESD5V0U1BA"
 			(at 0.1 1.9 0)
 			(layer "F.Fab")
@@
 	(footprint "fp:PinHeader_1x01"
 		(layer "F.Cu")
-		(at -10 5)
+		(at 10 5)
 		(descr "Through hole straight pin header, 1x03, 1.00mm pitch, single row")
 		(tags "Through hole pin header THT 1x03 1.00mm single row")
@@
 			)
 		)
-		(property "Value" "RUN"
+		(property "Value" "VCC"
 			(at 2 0.095 0)
 			(unlocked yes)
@@
 			)
 		)
-		(property "Value" "CESD5V0D5"
+		(property "Value" "DESD5V0U1BA"
 			(at 0.1 1.9 0)
 			(layer "F.Fab")
@@
 	(footprint "fp:PinHeader_1x01"
 		(layer "F.Cu")
-		(at -15 5)
+		(at 15 5)
 		(descr "Through hole straight pin header, 1x03, 1.00mm pitch, single row")
 		(tags "Through hole pin header THT 1x03 1.00mm single row")
@@
 	(footprint "fp:PinHeader_1x01"
 		(layer "F.Cu")
-		(at -5 5)
+		(at 5 5)
 		(descr "Through hole straight pin header, 1x03, 1.00mm pitch, single row")
 		(tags "Through hole pin header THT 1x03 1.00mm single row")
@@
 	(footprint "fp:PinHeader_1x01"
 		(layer "F.Cu")
-		(at 15 5)
+		(at -15 5)
 		(descr "Through hole straight pin header, 1x03, 1.00mm pitch, single row")
 		(tags "Through hole pin header THT 1x03 1.00mm single row")
@@
 			(layers "F.Cu" "F.Paste" "F.Mask")
 			(roundrect_rratio 0.2)
-			(net 9 "/COL_{0}")
+			(net 15 "/COL_{6}")
 			(pinfunction "P12")
 			(pintype "passive")
@@
 			(layers "F.Cu" "F.Paste" "F.Mask")
 			(roundrect_rratio 0.2)
-			(net 13 "/COL_{1}")
+			(net 18 "/COL_{5}")
 			(pinfunction "P13")
 			(pintype "passive")
@@
 			(layers "F.Cu" "F.Paste" "F.Mask")
 			(roundrect_rratio 0.2)
-			(net 14 "/COL_{2}")
+			(net 17 "/COL_{4}")
 			(pinfunction "P14")
 			(pintype "passive")
@@
 			(layers "F.Cu" "F.Paste" "F.Mask")
 			(roundrect_rratio 0.2)
-			(net 17 "/COL_{4}")
+			(net 14 "/COL_{2}")
 			(pinfunction "P16")
 			(pintype "passive")
@@
 			(layers "F.Cu" "F.Paste" "F.Mask")
 			(roundrect_rratio 0.2)
-			(net 18 "/COL_{5}")
+			(net 13 "/COL_{1}")
 			(pinfunction "P17")
 			(pintype "passive")
@@
 			(layers "F.Cu" "F.Paste" "F.Mask")
 			(roundrect_rratio 0.2)
-			(net 15 "/COL_{6}")
+			(net 9 "/COL_{0}")
 			(pinfunction "P18")
 			(pintype "passive")
@@
 	)
 	(gr_text "C0"
-		(at -15 3 0)
+		(at 15 3 0)
 		(layer "F.SilkS")
 		(effects
@@
 	)
 	(gr_text "C1"
-		(at -10 3 0)
+		(at 10 3 0)
 		(layer "F.SilkS")
 		(effects
@@
 	)
 	(gr_text "C2"
-		(at -5 3 0)
+		(at 5 3 0)
 		(layer "F.SilkS")
 		(effects
@@
 	)
 	(gr_text "C6"
-		(at 15 3 0)
+		(at -15 3 0)
 		(layer "F.SilkS")
 		(effects
@@
 	)
 	(gr_text "C5"
-		(at 10 3 0)
+		(at -10 3 0)
 		(layer "F.SilkS")
 		(effects
@@
 	)
 	(gr_text "C4"
-		(at 5 3 0)
+		(at -5 3 0)
 		(layer "F.SilkS")
 		(effects
@@
 	)
 	(segment
-		(start 4.9 -19.1)
-		(end 3.89 -19.1)
+		(start 11 -19.7)
+		(end 13.32 -17.38)
 		(width 0.1524)
 		(layer "F.Cu")
@@
 	)
 	(segment
-		(start -15 -0.21)
-		(end -15 5)
+		(start 11 -20)
+		(end 11 -19.7)
 		(width 0.1524)
 		(layer "F.Cu")
@@
 	)
 	(segment
-		(start 3.89 -19.1)
-		(end -15 -0.21)
+		(start 13.32 3.32)
+		(end 15 5)
+		(width 0.1524)
+		(layer "F.Cu")
+		(net 9)
+	)
+	(segment
+		(start 13.32 -17.38)
+		(end 13.32 3.32)
 		(width 0.1524)
 		(layer "F.Cu")
@@
 	)
 	(segment
-		(start 5.3 -18.57)
-		(end 4.96 -18.23)
-		(width 0.1524)
-		(layer "F.Cu")
-		(net 13)
-	)
-	(segment
-		(start -10 -4.06)
-		(end -10 5)
+		(start 10.1 -19.1)
+		(end 10.72 -19.1)
 		(width 0.1524)
 		(layer "F.Cu")
@@
 	)
 	(segment
-		(start 4.96 -18.23)
-		(end 4.17 -18.23)
+		(start 12.61 2.39)
+		(end 10 5)
 		(width 0.1524)
 		(layer "F.Cu")
@@
 	)
 	(segment
-		(start 5.3 -19.1)
-		(end 5.3 -18.57)
+		(start 10.72 -19.1)
+		(end 12.61 -17.21)
 		(width 0.1524)
 		(layer "F.Cu")
@@
 	)
 	(segment
-		(start 4.17 -18.23)
-		(end -10 -4.06)
+		(start 12.61 -17.21)
+		(end 12.61 2.39)
 		(width 0.1524)
 		(layer "F.Cu")
@@
 	)
 	(segment
-		(start 4.6 -17.73)
-		(end -5 -8.13)
+		(start 9.7 -18.57)
+		(end 10.11 -18.16)
 		(width 0.1524)
 		(layer "F.Cu")
@@
 	)
 	(segment
-		(start 5.7 -18.38)
-		(end 5.05 -17.73)
+		(start 11.06 -18.16)
+		(end 11.99 -17.23)
 		(width 0.1524)
 		(layer "F.Cu")
@@
 	)
 	(segment
-		(start 5.05 -17.73)
-		(end 4.6 -17.73)
+		(start 11.99 -1.99)
+		(end 5 5)
 		(width 0.1524)
 		(layer "F.Cu")
@@
 	)
 	(segment
-		(start 5.7 -19.1)
-		(end 5.7 -18.38)
+		(start 11.99 -17.23)
+		(end 11.99 -1.99)
 		(width 0.1524)
 		(layer "F.Cu")
@@
 	)
 	(segment
-		(start -5 -8.13)
-		(end -5 5)
+		(start 9.7 -19.1)
+		(end 9.7 -18.57)
 		(width 0.1524)
 		(layer "F.Cu")
@@
 	)
 	(segment
-		(start 11 -19.7)
-		(end 13.32 -17.38)
+		(start 10.11 -18.16)
+		(end 11.06 -18.16)
 		(width 0.1524)
 		(layer "F.Cu")
-		(net 15)
+		(net 14)
 	)
 	(segment
-		(start 11 -20)
-		(end 11 -19.7)
+		(start 4.9 -19.1)
+		(end 3.89 -19.1)
 		(width 0.1524)
 		(layer "F.Cu")
@@
 	)
 	(segment
-		(start 13.32 3.32)
-		(end 15 5)
+		(start -15 -0.21)
+		(end -15 5)
 		(width 0.1524)
 		(layer "F.Cu")
@@
 	)
 	(segment
-		(start 13.32 -17.38)
-		(end 13.32 3.32)
+		(start 3.89 -19.1)
+		(end -15 -0.21)
 		(width 0.1524)
 		(layer "F.Cu")
@@
 	)
 	(segment
-		(start 9.7 -18.57)
-		(end 10.11 -18.16)
+		(start 4.6 -17.73)
+		(end -5 -8.13)
 		(width 0.1524)
 		(layer "F.Cu")
@@
 	)
 	(segment
-		(start 11.06 -18.16)
-		(end 11.99 -17.23)
+		(start 5.7 -18.38)
+		(end 5.05 -17.73)
 		(width 0.1524)
 		(layer "F.Cu")
@@
 	)
 	(segment
-		(start 11.99 -1.99)
-		(end 5 5)
+		(start 5.05 -17.73)
+		(end 4.6 -17.73)
 		(width 0.1524)
 		(layer "F.Cu")
@@
 	)
 	(segment
-		(start 11.99 -17.23)
-		(end 11.99 -1.99)
+		(start 5.7 -19.1)
+		(end 5.7 -18.38)
 		(width 0.1524)
 		(layer "F.Cu")
@@
 	)
 	(segment
-		(start 9.7 -19.1)
-		(end 9.7 -18.57)
+		(start -5 -8.13)
+		(end -5 5)
 		(width 0.1524)
 		(layer "F.Cu")
@@
 	)
 	(segment
-		(start 10.11 -18.16)
-		(end 11.06 -18.16)
+		(start 5.3 -18.57)
+		(end 4.96 -18.23)
 		(width 0.1524)
 		(layer "F.Cu")
-		(net 17)
+		(net 18)
 	)
 	(segment
-		(start 10.1 -19.1)
-		(end 10.72 -19.1)
+		(start -10 -4.06)
+		(end -10 5)
 		(width 0.1524)
 		(layer "F.Cu")
@@
 	)
 	(segment
-		(start 12.61 2.39)
-		(end 10 5)
+		(start 4.96 -18.23)
+		(end 4.17 -18.23)
 		(width 0.1524)
 		(layer "F.Cu")
@@
 	)
 	(segment
-		(start 10.72 -19.1)
-		(end 12.61 -17.21)
+		(start 5.3 -19.1)
+		(end 5.3 -18.57)
 		(width 0.1524)
 		(layer "F.Cu")
@@
 	)
 	(segment
-		(start 12.61 -17.21)
-		(end 12.61 2.39)
+		(start 4.17 -18.23)
+		(end -10 -4.06)
 		(width 0.1524)
 		(layer "F.Cu")
