File: kicad/amosis_rhs.kicad_pcb (KiCad board)
At the start: 2 copper layers, 60 x 90 mm, 87 parts, among them J1 USB-C-16, J2 USB-C-16, J3 VALVE, M1 GND, M2 GND, M3 GND, Q1 MMBT3904, SW22 RESET, SW23 BOOT, U1 MIC5504-3.3YM5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

Commit message: logic & fixes
Parts:
- D25, D26: value CESD5V0D5 -> DESD5V0U1BA
- moved COL_{0}1 30.0 mm to (10.0, 5.00)
- moved COL_{6}1 30.0 mm to (-20.0, 5.00)
- moved COL_{1}1 20.0 mm to (5.00, 5.00)
- moved COL_{5}1 20.0 mm to (-15.0, 5.00)
- moved COL_{2}1 10.0 mm to (0.00, 5.00)
- moved COL_{4}1 10.0 mm to (-10.0, 5.00)
Connections:
- U3 pad 12: /COL_{0} -> /COL_{6}
- U3 pad 13: /COL_{1} -> /COL_{5}
- U3 pad 14: /COL_{2} -> /COL_{4}
- U3 pad 16: /COL_{4} -> /COL_{2}
- U3 pad 17: /COL_{5} -> /COL_{1}
- U3 pad 18: /COL_{6} -> /COL_{0}
Routing:
- net /COL_{6}: track 40.2 -> 29.3 mm
- net /COL_{0}: track 29.3 -> 40.2 mm
- net /COL_{5}: track 37.2 -> 26.7 mm
- net /COL_{1}: track 26.7 -> 37.2 mm
- net /COL_{4}: track 33.4 -> 27.1 mm
- net /COL_{2}: track 27.1 -> 33.4 mm
