File: kicad/amosis_rhs.kicad_sch (KiCad schematic)
At the start: 129 parts, among them J1 USB-C-16, J2 USB-C-16, J3 VALVE, M1 GND, M2 GND, M3 GND, Q1 MMBT3904, SW22 RESET, SW23 BOOT, U1 MIC5504-3.3YM5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

Commit message: logic & fixes
Parts:
- D25, D26: value CESD5V0D5 -> DESD5V0U1BA
- R10, R15: value 10 -> 24.9
- R14, R9: value 120 -> 49.9
Connections:
- net COL_{0}: now also D1.1 (K), D15.1 (K), D8.1 (K), U3.18 (P15); no longer D14.1 (K), D21.1 (K), D7.1 (K), U3.12 (P9)
- net COL_{1}: now also D16.1 (K), D2.1 (K), D9.1 (K), U3.17 (P14); no longer D13.1 (K), D20.1 (K), D6.1 (K), U3.13 (P10)
- net COL_{2}: now also D10.1 (K), D17.1 (K), D3.1 (K), U3.16 (P13); no longer D12.1 (K), D19.1 (K), D5.1 (K), U3.14 (P11)
- net COL_{4}: now also D12.1 (K), D19.1 (K), D5.1 (K), U3.14 (P11); no longer D10.1 (K), D17.1 (K), D3.1 (K), U3.16 (P13)
- net COL_{5}: now also D13.1 (K), D20.1 (K), D6.1 (K), U3.13 (P10); no longer D16.1 (K), D2.1 (K), D9.1 (K), U3.17 (P14)
- net COL_{6}: now also D14.1 (K), D21.1 (K), D7.1 (K), U3.12 (P9); no longer D1.1 (K), D15.1 (K), D8.1 (K), U3.18 (P15)
Other:
- moved on the sheet: COL_{0}1, COL_{1}1, COL_{2}1, COL_{3}1, COL_{4}1, COL_{5}1, COL_{6}1
Changed lines of the file:
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@@
 	(wire
 		(pts
-			(xy 179.07 185.42) (xy 186.69 185.42)
+			(xy 179.07 180.34) (xy 186.69 180.34)
 		)
 		(stroke
@@
 	(wire
 		(pts
-			(xy 179.07 190.5) (xy 186.69 190.5)
+			(xy 179.07 175.26) (xy 186.69 175.26)
 		)
 		(stroke
@@
 	(wire
 		(pts
-			(xy 179.07 175.26) (xy 186.69 175.26)
+			(xy 179.07 190.5) (xy 186.69 190.5)
 		)
 		(stroke
@@
 	(wire
 		(pts
-			(xy 179.07 187.96) (xy 186.69 187.96)
+			(xy 179.07 177.8) (xy 186.69 177.8)
 		)
 		(stroke
@@
 	(wire
 		(pts
-			(xy 179.07 177.8) (xy 186.69 177.8)
+			(xy 179.07 187.96) (xy 186.69 187.96)
 		)
 		(stroke
@@
 	(wire
 		(pts
-			(xy 179.07 180.34) (xy 186.69 180.34)
+			(xy 179.07 185.42) (xy 186.69 185.42)
 		)
 		(stroke
@@
 	)
 	(label "COL_{5}"
-		(at 186.69 187.96 180)
+		(at 186.69 177.8 180)
 		(fields_autoplaced yes)
 		(effects
@@
 	)
 	(label "COL_{4}"
-		(at 186.69 185.42 180)
+		(at 186.69 180.34 180)
 		(fields_autoplaced yes)
 		(effects
@@
 	)
 	(label "COL_{4}"
-		(at 255.27 91.44 180)
+		(at 255.27 86.36 180)
 		(fields_autoplaced yes)
 		(effects
@@
 	)
 	(label "COL_{6}"
-		(at 255.27 96.52 180)
+		(at 255.27 81.28 180)
 		(fields_autoplaced yes)
 		(effects
@@
 	)
 	(label "COL_{0}"
-		(at 255.27 81.28 180)
+		(at 255.27 96.52 180)
 		(fields_autoplaced yes)
 		(effects
@@
 	)
 	(label "COL_{1}"
-		(at 255.27 83.82 180)
+		(at 255.27 93.98 180)
 		(fields_autoplaced yes)
 		(effects
@@
 	)
 	(label "COL_{1}"
-		(at 186.69 177.8 180)
+		(at 186.69 187.96 180)
 		(fields_autoplaced yes)
 		(effects
@@
 	)
 	(label "COL_{2}"
-		(at 255.27 86.36 180)
+		(at 255.27 91.44 180)
 		(fields_autoplaced yes)
 		(effects
@@
 	)
 	(label "COL_{2}"
-		(at 186.69 180.34 180)
+		(at 186.69 185.42 180)
 		(fields_autoplaced yes)
 		(effects
@@
 	)
 	(label "COL_{5}"
-		(at 255.27 93.98 180)
+		(at 255.27 83.82 180)
 		(fields_autoplaced yes)
 		(effects
@@
 	)
 	(label "COL_{6}"
-		(at 186.69 190.5 180)
+		(at 186.69 175.26 180)
 		(fields_autoplaced yes)
 		(effects
@@
 	)
 	(label "COL_{0}"
-		(at 186.69 175.26 180)
+		(at 186.69 190.5 180)
 		(fields_autoplaced yes)
 		(effects
@@
 			)
 		)
-		(property "Value" "10"
-			(at 124.46 210.82 90)
+		(property "Value" "24.9"
+			(at 123.444 210.82 90)
 			(do_not_autoplace yes)
 			(effects
@@
 			)
 		)
-		(property "Value" "120"
-			(at 123.698 177.8 90)
+		(property "Value" "49.9"
+			(at 123.444 177.8 90)
 			(do_not_autoplace yes)
 			(effects
@@
 			)
 		)
-		(property "Value" "10"
-			(at 124.46 182.88 90)
+		(property "Value" "24.9"
+			(at 123.444 182.88 90)
 			(do_not_autoplace yes)
 			(effects
@@
 	(symbol
 		(lib_id "amosis:Conn_01x01_Socket")
-		(at 173.99 175.26 180)
+		(at 173.99 190.5 0)
+		(mirror y)
 		(unit 1)
 		(exclude_from_sim no)
@@
 		(dnp no)
 		(property "Reference" "COL_{0}1"
-			(at 173.355 175.26 0)
+			(at 173.355 190.5 0)
 			(do_not_autoplace yes)
 			(effects
@@
 		)
 		(property "Value" "COL_{0}"
-			(at 173.99 172.72 0)
+			(at 173.99 193.04 0)
 			(effects
 				(font
@@
 		)
 		(property "Footprint" "fp:PinHeader_1x01"
-			(at 173.99 175.26 0)
+			(at 173.99 190.5 0)
 			(effects
 				(font
@@
 		)
 		(property "Datasheet" "~"
-			(at 173.99 175.26 0)
+			(at 173.99 190.5 0)
 			(effects
 				(font
@@
 		)
 		(property "Description" "Generic connector, single row, 01x01, script generated"
-			(at 173.99 175.26 0)
+			(at 173.99 190.5 0)
 			(effects
 				(font
@@
 	(symbol
 		(lib_id "amosis:Conn_01x01_Socket")
-		(at 173.99 177.8 180)
+		(at 173.99 187.96 0)
+		(mirror y)
 		(unit 1)
 		(exclude_from_sim no)
@@
 		(dnp no)
 		(property "Reference" "COL_{1}1"
-			(at 173.355 177.8 0)
+			(at 173.355 187.96 0)
 			(do_not_autoplace yes)
 			(effects
@@
 		)
 		(property "Value" "COL_{1}"
-			(at 173.99 175.26 0)
+			(at 173.99 190.5 0)
 			(effects
 				(font
@@
 		)
 		(property "Footprint" "fp:PinHeader_1x01"
-			(at 173.99 177.8 0)
+			(at 173.99 187.96 0)
 			(effects
 				(font
@@
 		)
 		(property "Datasheet" "~"
-			(at 173.99 177.8 0)
+			(at 173.99 187.96 0)
 			(effects
 				(font
@@
 		)
 		(property "Description" "Generic connector, single row, 01x01, script generated"
-			(at 173.99 177.8 0)
+			(at 173.99 187.96 0)
 			(effects
 				(font
@@
 			)
 		)
-		(property "Value" "120"
-			(at 123.698 205.74 90)
+		(property "Value" "49.9"
+			(at 123.444 205.74 90)
 			(do_not_autoplace yes)
 			(effects
@@
 	(symbol
 		(lib_id "amosis:Conn_01x01_Socket")
-		(at 173.99 190.5 180)
+		(at 173.99 175.26 0)
+		(mirror y)
 		(unit 1)
 		(exclude_from_sim no)
@@
 		(dnp no)
 		(property "Reference" "COL_{6}1"
-			(at 173.355 190.5 0)
+			(at 173.355 175.26 0)
 			(do_not_autoplace yes)
 			(effects
@@
 		)
 		(property "Value" "ROW_{0}"
-			(at 173.99 187.96 0)
+			(at 173.99 177.8 0)
 			(effects
 				(font
@@
 		)
 		(property "Footprint" "fp:PinHeader_1x01"
-			(at 173.99 190.5 0)
+			(at 173.99 175.26 0)
 			(effects
 				(font
@@
 		)
 		(property "Datasheet" "~"
-			(at 173.99 190.5 0)
+			(at 173.99 175.26 0)
 			(effects
 				(font
@@
 		)
 		(property "Description" "Generic connector, single row, 01x01, script generated"
-			(at 173.99 190.5 0)
+			(at 173.99 175.26 0)
 			(effects
 				(font
@@
 	(symbol
 		(lib_id "amosis:Conn_01x01_Socket")
-		(at 173.99 187.96 180)
+		(at 173.99 177.8 0)
+		(mirror y)
 		(unit 1)
 		(exclude_from_sim no)
@@
 		(dnp no)
 		(property "Reference" "COL_{5}1"
-			(at 173.355 187.96 0)
+			(at 173.355 177.8 0)
 			(do_not_autoplace yes)
 			(effects
@@
 		)
 		(property "Value" "COL_{5}"
-			(at 173.99 185.42 0)
+			(at 173.99 180.34 0)
 			(effects
 				(font
@@
 		)
 		(property "Footprint" "fp:PinHeader_1x01"
-			(at 173.99 187.96 0)
+			(at 173.99 177.8 0)
 			(effects
 				(font
@@
 		)
 		(property "Datasheet" "~"
-			(at 173.99 187.96 0)
+			(at 173.99 177.8 0)
 			(effects
 				(font
@@
 		)
 		(property "Description" "Generic connector, single row, 01x01, script generated"
-			(at 173.99 187.96 0)
+			(at 173.99 177.8 0)
 			(effects
 				(font
@@
 	(symbol
 		(lib_id "amosis:Conn_01x01_Socket")
-		(at 173.99 185.42 180)
+		(at 173.99 180.34 0)
+		(mirror y)
 		(unit 1)
 		(exclude_from_sim no)
@@
 		(dnp no)
 		(property "Reference" "COL_{4}1"
-			(at 173.355 185.42 0)
+			(at 173.355 180.34 0)
 			(do_not_autoplace yes)
 			(effects
@@
 		)
 		(property "Footprint" "fp:PinHeader_1x01"
-			(at 173.99 185.42 0)
+			(at 173.99 180.34 0)
 			(effects
 				(font
@@
 		)
 		(property "Datasheet" "~"
-			(at 173.99 185.42 0)
+			(at 173.99 180.34 0)
 			(effects
 				(font
@@
 		)
 		(property "Description" "Generic connector, single row, 01x01, script generated"
-			(at 173.99 185.42 0)
+			(at 173.99 180.34 0)
 			(effects
 				(font
@@
 	(symbol
 		(lib_id "amosis:Conn_01x01_Socket")
-		(at 173.99 180.34 180)
+		(at 173.99 185.42 0)
+		(mirror y)
 		(unit 1)
 		(exclude_from_sim no)
@@
 		(dnp no)
 		(property "Reference" "COL_{2}1"
-			(at 173.355 180.34 0)
+			(at 173.355 185.42 0)
 			(do_not_autoplace yes)
 			(effects
@@
 		)
 		(property "Value" "COL_{2}"
-			(at 173.99 177.8 0)
+			(at 173.99 187.96 0)
 			(effects
 				(font
@@
 		)
 		(property "Footprint" "fp:PinHeader_1x01"
-			(at 173.99 180.34 0)
+			(at 173.99 185.42 0)
 			(effects
 				(font
@@
 		)
 		(property "Datasheet" "~"
-			(at 173.99 180.34 0)
+			(at 173.99 185.42 0)
 			(effects
 				(font
@@
 		)
 		(property "Description" "Generic connector, single row, 01x01, script generated"
-			(at 173.99 180.34 0)
+			(at 173.99 185.42 0)
 			(effects
 				(font
@@
 	(symbol
 		(lib_id "amosis:Conn_01x01_Socket")
-		(at 173.99 182.88 180)
+		(at 173.99 182.88 0)
+		(mirror y)
 		(unit 1)
 		(exclude_from_sim no)
@@
 		)
 		(property "Value" "COL_{3}"
-			(at 173.99 180.34 0)
+			(at 173.99 185.42 0)
 			(effects
 				(font
@@
 			)
 		)
-		(property "Value" "CESD5V0D5"
+		(property "Value" "DESD5V0U1BA"
 			(at 85.725 167.64 0)
 			(do_not_autoplace yes)
@@
 			)
 		)
-		(property "Value" "CESD5V0D5"
+		(property "Value" "DESD5V0U1BA"
 			(at 100.965 167.64 0)
 			(do_not_autoplace yes)
